File: v1/fun-size.sch (KiCad schematic (older format))
At the start: 80 parts, among them J1 MJ-4PP-9, J2 MJ-4PP-9, SW1 SW_PUSH, SW10 SW_PUSH, SW11 SW_PUSH, SW12 SW_PUSH, SW13 SW_PUSH, SW14 SW_PUSH, SW15 SW_PUSH, SW16 SW_PUSH, SW17 SW_PUSH, SW18 SW_PUSH, SW19 SW_PUSH, SW2 SW_PUSH, SW20 SW_PUSH, SW21 SW_PUSH, SW22 SW_PUSH, SW23 SW_PUSH, SW24 SW_PUSH, SW25 SW_PUSH, SW26 SW_PUSH, SW27 SW_PUSH, SW28 SW_PUSH, SW29 SW_PUSH, SW3 SW_PUSH, SW30 SW_PUSH, SW31 SW_PUSH, SW32 SW_PUSH, SW33 SW_PUSH, SW34 SW_PUSH, SW35 SW_PUSH, SW36 SW_PUSH, SW37 Rotary_Encoder_Switch, SW38 Rotary_Encoder_Switch, SW4 SW_PUSH, SW5 SW_PUSH, SW6 SW_PUSH, SW7 SW_PUSH, SW8 SW_PUSH, SW9 SW_PUSH, U1 ProMicro, U2 ProMicro

Commit message: add mounting holes for a case
Parts:
- added SW39, SW40: Rotary_Encoder_Switch, Encoder:RollerEncoder_Panasonic_EVQWGD001, symbol Device:Rotary_Encoder_Switch
Connections:
- net COL_L_1: now also U1.16 (B1/15); no longer U1.19 (F5/A2)
- net COL_L_2: now also U1.17 (F7/A0); no longer U1.18 (F6/A1)
- net COL_L_3: now also SW38.S1, U1.18 (F6/A1); no longer U1.17 (F7/A0)
- net COL_L_4: now also U1.19 (F5/A2); no longer U1.16 (B1/15)
- net COL_L_5: now also SW37.S1, U1.20 (F4/A3); no longer SW38.S1, U1.15 (B3/14)
- net COL_R_1: now also U2.5 (2/D1/SDA), SW39.S1; no longer SW37.S1, U2.15 (B3/14)
- net COL_R_2: now also U2.6 (3/D0/SCL); no longer U2.16 (B1/15)
- net COL_R_3: now also U2.7 (4/D4), SW40.S1; no longer U2.17 (F7/A0)
- net COL_R_4: now also U2.8 (5/C6); no longer U2.18 (F6/A1)
- net COL_R_5: now also U2.9 (6/D7); no longer U2.19 (F5/A2)
- net ROW_L_1: now also U1.5 (2/D1/SDA); no longer U1.7 (4/D4)
- net ROW_L_2: now also U1.6 (3/D0/SCL); no longer U1.8 (5/C6)
- net ROW_L_3: now also U1.7 (4/D4); no longer U1.9 (6/D7)
- net ROW_L_4: now also U1.8 (5/C6); no longer U1.10 (7/E6)
- net ROW_R_1: now also U2.20 (F4/A3); no longer U2.7 (4/D4)
- net ROW_R_2: now also U2.19 (F5/A2); no longer U2.8 (5/C6)
- net ROW_R_3: now also U2.18 (F6/A1); no longer U2.9 (6/D7)
- net ROW_R_4: now also U2.17 (F7/A0); no longer U2.10 (7/E6)
- net ENC_L_B_2: now reaches U1.14 (B2/16)
- net ENC_L_B_2: now also SW38.B
- net ENC_L_2_OUT: now reaches D16.2 (A), SW16.2
- net ENC_L_2_OUT: now also SW38.S2
- net ENC_R_B_1: now reaches U2.14 (B2/16)
- net ENC_R_B_1: now also SW39.B
- net ENC_R_2_OUT: now reaches D34.2 (A), SW34.2
- net ENC_R_2_OUT: now also SW40.S2
- net ENC_L_A renamed ENC_L_A_2
- net ENC_L_A_2: now also U1.13 (B6/10); no longer U1.11 (8/B4)
- net ENC_L_B renamed ENC_L_A_1
- net ENC_L_A_1: now also SW37.A; no longer SW38.B
- net ENC_L_C renamed ENC_L_C_2
- net ENC_L_C_2: now also U1.15 (B3/14); no longer U1.13 (B6/10)
- net ENC_L_OUT renamed ENC_L_1_OUT
- net ENC_L_1_OUT: now also SW37.S2; no longer SW38.S2
- net ENC_R_A renamed ENC_R_B_2
- net ENC_R_B_2: now also SW40.B; no longer SW37.A
- net ENC_R_B renamed ENC_L_B_1
- net ENC_L_B_1: now also U1.11 (8/B4); no longer U2.12 (9/B5)
- net ENC_R_C renamed ENC_L_C_1
- net ENC_L_C_1: now also U1.10 (7/E6); no longer U2.13 (B6/10)
- net ENC_R_OUT renamed ENC_R_1_OUT
- net ENC_R_1_OUT: now also SW39.S2; no longer SW37.S2
- new net ENC_R_A_1: SW39.A, U2.15 (B3/14)
- new net ENC_R_A_2: SW40.A, U2.10 (7/E6)
- new net ENC_R_C_1: SW39.C, U2.13 (B6/10)
- new net ENC_R_C_2: SW40.C, U2.12 (9/B5)
- no-connect marks 14 -> 8
Other:
- moved on the sheet: SW37, SW38
