File: v1/fun-size.kicad_pcb (KiCad board)
At the start: 2 copper layers, 13.3 x 9 mm, 80 parts, among them J1 MJ-4PP-9, J2 MJ-4PP-9, SW1 SW_PUSH, SW10 SW_PUSH, SW11 SW_PUSH, SW12 SW_PUSH, SW13 SW_PUSH, SW14 SW_PUSH, SW15 SW_PUSH, SW16 SW_PUSH, SW17 SW_PUSH, SW18 SW_PUSH, SW19 SW_PUSH, SW2 SW_PUSH, SW20 SW_PUSH, SW21 SW_PUSH, SW22 SW_PUSH, SW23 SW_PUSH, SW24 SW_PUSH, SW25 SW_PUSH, SW26 SW_PUSH, SW27 SW_PUSH, SW28 SW_PUSH, SW29 SW_PUSH, SW3 SW_PUSH, SW30 SW_PUSH, SW31 SW_PUSH, SW32 SW_PUSH, SW33 SW_PUSH, SW34 SW_PUSH, SW35 SW_PUSH, SW36 SW_PUSH, SW37 Rotary_Encoder_Switch, SW38 Rotary_Encoder_Switch, SW4 SW_PUSH, SW5 SW_PUSH, SW6 SW_PUSH, SW7 SW_PUSH, SW8 SW_PUSH, SW9 SW_PUSH, U1 ProMicro, U2 ProMicro

Commit message: finish PCB design v1
Parts:
- moved SW38 0.20 mm to (137.2, 106.7)
- moved D18 0.20 mm to (128.3, 88.3)
- moved J1 0.20 mm to (148.3, 86.2)
- moved SW18 0.20 mm to (136.9, 106.2)
- moved SWRST1 0.20 mm to (128.3, 85.1)
- moved U1 0.20 mm to (134.3, 66.1)
- moved D10 0.20 mm to (111.9, 49.8)
- moved D11 0.20 mm to (37.8, 83.5)
- moved D12 0.20 mm to (53.5, 63.4)
- moved D13 0.20 mm to (72.1, 59.1)
- moved D14 0.20 mm to (91.7, 64.1)
- moved D15 0.20 mm to (109.5, 66.6)
- moved D16 0.20 mm to (101.1, 87.8)
- moved D17 0.20 mm to (120.9, 93.2)
- moved D3 0.20 mm to (72.1, 25.1)
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Routing:
- net ROW_L_1: track 159.9 -> 161.6 mm
- net ENC_L_A: track 30.0 -> 30.6 mm
- net COL_L_5: track 125.9 -> 126.4 mm
Other:
- board size 13.3 x 9 mm -> 263.6 x 105.5 mm
- net class Default: clearance 0.2 -> 0.199
- rule trace_clearance: 0.2 -> 0.199
- board text added: "By S'mores"
- board text added: "Fun"
- board text added: "Fun Size v1"
- board text added: "Size"

Commit message: add mounting holes for a case
Parts:
- added Ref**: Val**, kbd:M2_HOLE_v3, F.Cu at (155.7, 122.1)
- added Ref**: Val**, kbd:M2_HOLE_v3, F.Cu at (38.6, 69.4)
- added Ref**: Val**, kbd:M2_HOLE_v3, F.Cu at (142.0, 122.1)
- added Ref**: Val**, kbd:M2_HOLE_v3, F.Cu at (120.4, 80.8)
- added Ref**: Val**, kbd:M2_HOLE_v3, F.Cu at (177.9, 80.8)
- added Ref**: Val**, kbd:M2_HOLE_v3, F.Cu at (210.7, 114.5)
- added Ref**: Val**, kbd:M2_HOLE_v3, F.Cu at (247.9, 114.5)
- added Ref**: Val**, kbd:M2_HOLE_v3, F.Cu at (260.1, 69.4)
- added Ref**: Val**, kbd:M2_HOLE_v3, F.Cu at (216.8, 70.1)
- added Ref**: Val**, kbd:M2_HOLE_v3, F.Cu at (86.6, 114.3)
- added Ref**: Val**, kbd:M2_HOLE_v3, F.Cu at (81.5, 70.2)
- added Ref**: Val**, kbd:M2_HOLE_v3, F.Cu at (51.6, 114.4)
- added SW39: Rotary_Encoder_Switch, Encoder:RollerEncoder_Panasonic_EVQWGD001, F.Cu at (163.0, 134.2)
- added SW40: Rotary_Encoder_Switch, Encoder:RollerEncoder_Panasonic_EVQWGD001, F.Cu at (199.7, 121.0)
- moved D34 42.0 mm to (166.9, 114.8), turned to 180 degrees
- moved SW38 40.2 mm to (99.7, 121.0), turned to 260 degrees
- moved SW37 39.7 mm to (136.2, 134.6), turned to 240 degrees
- moved D16 39.1 mm to (131.2, 112.8), turned to 180 degrees
- moved SWRST1 28.9 mm to (126.2, 113.9), turned to 90 degrees
- moved SWRST2 28.6 mm to (172.0, 113.6), turned to 90 degrees
- moved D19 27.9 mm to (271.0, 78.5)
- moved D24 27.9 mm to (266.3, 94.9)
- moved D25 27.9 mm to (247.1, 74.3)
- moved D26 27.9 mm to (227.0, 69.9)
- moved D29 27.9 mm to (261.8, 111.3)
- moved D31 27.9 mm to (227.0, 86.9)
- moved SW13 27.9 mm to (71.3, 92.0)
- moved SW16 27.9 mm to (99.2, 120.6)
- moved SW18 27.9 mm to (135.9, 134.1)
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Connections:
- net Net-(D34-Pad2) renamed ENC_R_2_OUT
- D16 pad 2: Net-(D16-Pad2) -> ENC_L_2_OUT
- D18 pad 2: ENC_L_OUT -> ENC_L_1_OUT
- D36 pad 2: ENC_R_OUT -> ENC_R_1_OUT
- SW16 pad 2: Net-(D16-Pad2) -> ENC_L_2_OUT
- SW18 pad 2: ENC_L_OUT -> ENC_L_1_OUT
- SW36 pad 2: ENC_R_OUT -> ENC_R_1_OUT
- SW37 pad A: ENC_R_A -> ENC_L_A_1
- SW37 pad B: ENC_R_B -> ENC_L_B_1
- SW37 pad C: ENC_R_C -> ENC_L_C_1
- SW37 pad S1: COL_R_1 -> COL_L_5
- SW37 pad S2: ENC_R_OUT -> ENC_L_1_OUT
- SW38 pad A: ENC_L_A -> ENC_L_A_2
- SW38 pad B: ENC_L_B -> ENC_L_B_2
- SW38 pad C: ENC_L_C -> ENC_L_C_2
- SW38 pad S1: COL_L_5 -> COL_L_3
- SW38 pad S2: ENC_L_OUT -> ENC_L_2_OUT
- U1 pad 10: ROW_L_4 -> ENC_L_C_1
- U1 pad 11: ENC_L_A -> ENC_L_B_1
- U1 pad 12: ENC_L_B -> ENC_L_A_1
- U1 pad 13: ENC_L_C -> ENC_L_A_2
- U1 pad 14: Net-(U1-Pad14) -> ENC_L_B_2
- U1 pad 15: COL_L_5 -> ENC_L_C_2
- U1 pad 16: COL_L_4 -> COL_L_1
- U1 pad 17: COL_L_3 -> COL_L_2
- U1 pad 18: COL_L_2 -> COL_L_3
- U1 pad 19: COL_L_1 -> COL_L_4
- U1 pad 20: Net-(U1-Pad20) -> COL_L_5
- U1 pad 5: Net-(U1-Pad5) -> ROW_L_1
- U1 pad 6: Net-(U1-Pad6) -> ROW_L_2
- U1 pad 7: ROW_L_1 -> ROW_L_3
- U1 pad 8: ROW_L_2 -> ROW_L_4
- U1 pad 9: ROW_L_3 -> Net-(U1-Pad9)
- U2 pad 10: ROW_R_4 -> ENC_R_A_2
- U2 pad 11: ENC_R_A -> ENC_R_B_2
- U2 pad 12: ENC_R_B -> ENC_R_C_2
- U2 pad 13: ENC_R_C -> ENC_R_C_1
- U2 pad 14: Net-(U2-Pad14) -> ENC_R_B_1
- U2 pad 15: COL_R_1 -> ENC_R_A_1
- U2 pad 16: COL_R_2 -> Net-(U2-Pad16)
- U2 pad 17: COL_R_3 -> ROW_R_4
- U2 pad 18: COL_R_4 -> ROW_R_3
- U2 pad 19: COL_R_5 -> ROW_R_2
- U2 pad 20: Net-(U2-Pad20) -> ROW_R_1
- U2 pad 5: Net-(U2-Pad5) -> COL_R_1
- U2 pad 6: Net-(U2-Pad6) -> COL_R_2
- U2 pad 7: ROW_R_1 -> COL_R_3
- U2 pad 8: ROW_R_2 -> COL_R_4
- U2 pad 9: ROW_R_3 -> COL_R_5
Routing:
- net ENC_L_2_OUT: track 0.00 -> 46.1 mm
- net ENC_L_1_OUT: track 0.00 -> 44.5 mm, vias 0 -> 1
- net ENC_L_OUT: track 40.8 -> 0.00 mm, vias 1 -> 0
- net ROW_R_3: track 116.5 -> 156.3 mm
- net ENC_R_2_OUT: track 12.0 -> 51.7 mm
- net ENC_R_A_2: track 0.00 -> 37.3 mm
- net ENC_R_1_OUT: track 0.00 -> 36.6 mm
- net ENC_R_OUT: track 35.5 -> 0.00 mm, vias 1 -> 0
- net ENC_L_C_2: track 0.00 -> 33.6 mm
- net ENC_R_B_2: track 0.00 -> 32.8 mm
- net ENC_L_C: track 31.7 -> 0.00 mm, vias 2 -> 0
- net COL_R_4: track 151.5 -> 120.4 mm
- net ENC_R_B_1: track 0.00 -> 31.0 mm
- net ENC_L_C_1: track 0.00 -> 30.8 mm
- net ENC_R_A_1: track 0.00 -> 30.6 mm
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Other:
- board size 263.6 x 105.5 mm -> 262.2 x 101 mm
- net class Default: clearance 0.199 -> 0.2
- rule trace_clearance: 0.199 -> 0.2

Commit message: thicken bridges between halves
Routing:
- added copper zone on B.Cu, net (none)
- added copper zone on F.Cu, net (none)
Other:
- outline, holes or cut-outs redrawn
- rule trace_min: 0.2 -> 0.199
